Commit message: It finally works.I have included a gazebo file where you can have some fun. Enjoy!

File: description/robot_core.xacro (robot description, xacro)
@@ -1,50 +1,53 @@
 <?xml version="1.0"?>
-<robot xmlns:xacro="http://www.ros.org/wiki/xacro"  name="robot">
-    <xacro:include filename="inertial_macros.xacro" />
-    <material name = "white">
-        <color rgba="1 1 1 1 " />
+<robot xmlns:xacro="http://www.ros.org/wiki/xacro" >
+    <xacro:include filename="inertial_macros.xacro"/>
+    <material name="white">
+        <color rgba="1 1 1 1" />
     </material>
-    <material name = "orange">
-        <color rgba="1 0.3 0.1 1 " />
+    <material name="orange">
+        <color rgba="1 0.3 0.1 1"/>
     </material>
-    <material name = "blue">
-        <color rgba="0.2 0.2 1 1 " />
+    <material name="blue">
+        <color rgba="0.2 0.2 1 1"/>
     </material>
-    <material name = "black">
-        <color rgba="0 0 0 1 " />
+    <material name="black">
+        <color rgba="0 0 0 1"/>
     </material>
-    <!-- Base Link-->
+    <!-- BASE LINK -->
     <link name="base_link">
     </link>
-    <!-- Chassis Link-->
-    <joint name= "chassis_joint" type = "fixed" >
-        <parent link = "base_link"/>
-        <child link = "chassis"/>
-        <origin xyz = "-0.1 0 0"/>
+    <!-- CHASSIS LINK -->
+    <joint name="chassis_joint" type="fixed">
+        <parent link="base_link"/>
+        <child link="chassis"/>
+        <origin xyz="-0.1 0 0"/>
     </joint>
-    <link name= "chassis">
+    <link name="chassis">
         <visual>
-            <origin xyz = "0.15 0 0.075"/>
+            <origin xyz="0.15 0 0.075"/>
             <geometry>
-                <box size = "0.3 0.3 0.15"/>
+                <box size="0.3 0.3 0.15"/>
             </geometry>
-            <material name = "white"/>
+            <material name="white"/>
         </visual>
         <collision>
-            <origin xyz = "0.15 0 0.075"/>
+            <origin xyz="0.15 0 0.075"/>
             <geometry>
-                <box size = "0.3 0.3 0.15"/>
+                <box size="0.3 0.3 0.15"/>
             </geometry>
         </collision>
-        <xacro:inertial_box mass ="0.5" x="0.3" y="0.3" z="0.15">
+        <xacro:inertial_box mass="0.5" x="0.3" y="0.3" z="0.15">
             <origin xyz="0.15 0 0.075" rpy="0 0 0"/>
         </xacro:inertial_box>
     </link>
-    <!-- Left Wheel Link-->
-    <joint name="Left_wheel_joint" type="continuous">
-        <parent link="base_link" />
-        <child link="left_wheel" />
-        <origin xyz= "0 0.175 0" rpy="-${pi/2} 0 0"/>
-        <axis xyz="0.0 0.0 1.0"/>
+    <gazebo reference="chassis">
+        <material>Gazebo/White</material>
+    </gazebo>
+    <!-- LEFT WHEEL LINK -->
+    <joint name="left_wheel_joint" type="continuous">
+        <parent link="base_link"/>
+        <child link="left_wheel"/>
+        <origin xyz="0 0.175 0" rpy="-${pi/2} 0 0" />
+        <axis xyz="0 0 1"/>
     </joint>
     <link name="left_wheel">
@@ -53,5 +56,5 @@
                 <cylinder radius="0.05" length="0.04"/>
             </geometry>
-                <material name="blue"/>
+            <material name="blue"/>
         </visual>
         <collision>
@@ -64,10 +67,13 @@
         </xacro:inertial_cylinder>
     </link>
-    <!-- Right Wheel Link-->
+    <gazebo reference="left_wheel">
+        <material>Gazebo/Blue</material>
+    </gazebo>
+    <!-- RIGHT WHEEL LINK -->
     <joint name="right_wheel_joint" type="continuous">
-        <parent link="base_link" />
-        <child link="right_wheel" />
-        <origin xyz= "0 -0.175 0" rpy="${pi/2} 0 0"/>
-        <axis xyz="0.0 0.0 -1.0"/>
+        <parent link="base_link"/>
+        <child link="right_wheel"/>
+        <origin xyz="0 -0.175 0" rpy="${pi/2} 0 0" />
+        <axis xyz="0 0 -1"/>
     </joint>
     <link name="right_wheel">
@@ -76,5 +82,5 @@
                 <cylinder radius="0.05" length="0.04"/>
             </geometry>
-                <material name="blue"/>
+            <material name="blue"/>
         </visual>
         <collision>
@@ -87,5 +93,8 @@
         </xacro:inertial_cylinder>
     </link>
-    <!-- Caster Wheel Link-->
+    <gazebo reference="right_wheel">
+        <material>Gazebo/Blue</material>
+    </gazebo>
+    <!-- CASTER WHEEL LINK -->
     <joint name="caster_wheel_joint" type="fixed">
         <parent link="chassis"/>
@@ -109,3 +118,8 @@
         </xacro:inertial_sphere>
     </link>
+    <gazebo reference="caster_wheel">
+        <material>Gazebo/Black</material>
+        <mu1 value="0.001"/>
+        <mu2 value="0.001"/>
+    </gazebo>
 </robot>
